Commit message: launchfile changes and code fixes

File: Environment_config/GrGSL_RA-L_2021/navigation_config/resources/giraff.xacro (robot description, xacro)
@@ -1,4 +1,9 @@
-<?xml version="1.0"?>
-<robot name="giraff">
+<?xml version="1.0" ?>
+<!-- =================================================================================== -->
+<!-- |    This document was autogenerated by xacro from giraff.urdf                    | -->
+<!-- |    EDITING THIS FILE BY HAND IS NOT RECOMMENDED                                 | -->
+<!-- =================================================================================== -->
+<robot xmlns:xacro="http://www.ros.org/wiki/xacro" name="giraff">
+  <xacro:arg name="frame_ns" default="giraff"/>
   ### Define colors
   <material name="blue">
@@ -11,5 +16,5 @@
     <color rgba="1 1 1 1"/>
   </material>
-    <material name="grey">
+  <material name="grey">
     <color rgba="0.5 0.5 0.5 1"/>
   </material>
@@ -21,5 +26,5 @@
   </material>
   # Base
-  <link name="base_link">
+  <link name="$(arg frame_ns)_base_link">
     <visual>
       <geometry>
@@ -31,5 +36,5 @@
   </link>
   # Right wheel
-  <link name="right_wheel">
+  <link name="$(arg frame_ns)_right_wheel">
     <visual>
       <origin rpy="1.57075 0 0" xyz="0 0 0"/>
@@ -40,11 +45,11 @@
     </visual>
   </link>
-  <joint name="base_to_right_wheel_joint" type="fixed">
-    <parent link="base_link"/>
-    <child link="right_wheel"/>
+  <joint name="$(arg frame_ns)_base_to_right_wheel_joint" type="fixed">
+    <parent link="$(arg frame_ns)_base_link"/>
+    <child link="$(arg frame_ns)_right_wheel"/>
     <origin rpy="0 0 0" xyz="0 0.26 0.1"/>
   </joint>
   #Left wheel
-  <link name="left_wheel">
+  <link name="$(arg frame_ns)_left_wheel">
     <visual>
       <origin rpy="1.57075 0 0" xyz="0 0 0"/>
@@ -55,11 +60,11 @@
     </visual>
   </link>
-  <joint name="base_to_left_wheel_joint" type="fixed">
-    <parent link="base_link"/>
-    <child link="left_wheel"/>
+  <joint name="$(arg frame_ns)_base_to_left_wheel_joint" type="fixed">
+    <parent link="$(arg frame_ns)_base_link"/>
+    <child link="$(arg frame_ns)_left_wheel"/>
     <origin rpy="0 0 0" xyz="0 -0.26 0.1"/>
   </joint>
   # Body
-  <link name="body">
+  <link name="$(arg frame_ns)_body">
     <visual>
       <geometry>
@@ -69,11 +74,11 @@
     </visual>
   </link>
-  <joint name="base_to_body" type="fixed">
-    <parent link="base_link"/>
-    <child link="body"/>
+  <joint name="$(arg frame_ns)_base_to_body" type="fixed">
+    <parent link="$(arg frame_ns)_base_link"/>
+    <child link="$(arg frame_ns)_body"/>
     <origin xyz="0.0 0.0 0.455"/>
   </joint>
   #Neck
-  <link name="neck">
+  <link name="$(arg frame_ns)_neck">
     <visual>
       <geometry>
@@ -83,11 +88,11 @@
     </visual>
   </link>
-  <joint name="body_to_neck" type="fixed">
-    <parent link="body"/>
-    <child link="neck"/>
+  <joint name="$(arg frame_ns)_body_to_neck" type="fixed">
+    <parent link="$(arg frame_ns)_body"/>
+    <child link="$(arg frame_ns)_neck"/>
     <origin xyz="0.0 0.0 0.45"/>
   </joint>
   #Head
-  <link name="head">
+  <link name="$(arg frame_ns)_head">
     <visual>
       <geometry>
@@ -97,11 +102,11 @@
     </visual>
   </link>
-  <joint name="neck_to_head" type="fixed">
-    <parent link="neck"/>
-    <child link="head"/>
+  <joint name="$(arg frame_ns)_neck_to_head" type="fixed">
+    <parent link="$(arg frame_ns)_neck"/>
+    <child link="$(arg frame_ns)_head"/>
     <origin xyz="0 0 0.415"/>
   </joint>
   #Screen
-  <link name="screen">
+  <link name="$(arg frame_ns)_screen">
     <visual>
       <geometry>
@@ -111,12 +116,12 @@
     </visual>
   </link>
-  <joint name="head_to_screen" type="fixed">
-    <parent link="head"/>
-    <child link="screen"/>
+  <joint name="$(arg frame_ns)_head_to_screen" type="fixed">
+    <parent link="$(arg frame_ns)_head"/>
+    <child link="$(arg frame_ns)_screen"/>
     <origin xyz="0.02 0.0 0.0"/>
   </joint>
   ## EXTRAS ##
   #Hokuyo front
-  <link name="hokuyo_front">
+  <link name="$(arg frame_ns)_hokuyo_front">
     <visual>
       <geometry>
@@ -126,11 +131,11 @@
     </visual>
   </link>
-  <joint name="base_to_hokuyo_front" type="fixed">
-    <parent link="base_link"/>
-    <child link="hokuyo_front"/>
+  <joint name="$(arg frame_ns)_base_to_hokuyo_front" type="fixed">
+    <parent link="$(arg frame_ns)_base_link"/>
+    <child link="$(arg frame_ns)_hokuyo_front"/>
     <origin xyz="0.2 0.0 0.28"/>
   </joint>
   #red button
-  <link name="red_button">
+  <link name="$(arg frame_ns)_red_button">
     <visual>
       <geometry>
@@ -140,11 +145,11 @@
     </visual>
   </link>
-  <joint name="body_to_red_button" type="fixed">
-    <parent link="body"/>
-    <child link="red_button"/>
+  <joint name="$(arg frame_ns)_body_to_red_button" type="fixed">
+    <parent link="$(arg frame_ns)_body"/>
+    <child link="$(arg frame_ns)_red_button"/>
     <origin xyz="0.11 0.05 0.225"/>
   </joint>
   #green button
-  <link name="green_button">
+  <link name="$(arg frame_ns)_green_button">
     <visual>
       <geometry>
@@ -154,7 +159,7 @@
     </visual>
   </link>
-  <joint name="body_to_green_button" type="fixed">
-    <parent link="body"/>
-    <child link="green_button"/>
+  <joint name="$(arg frame_ns)_body_to_green_button" type="fixed">
+    <parent link="$(arg frame_ns)_body"/>
+    <child link="$(arg frame_ns)_green_button"/>
     <origin xyz="0.11 -0.05 0.225"/>
   </joint>
